File: PCB/LtDev.kicad_sch (KiCad schematic)
At the start: 112 parts, among them IC1 TMUX1134PWR, IC2 MMS9013-H-TP, IC3 TPS2116DRLR, IC4 TPS2116DRLR, J1 Conn_JTAG_02x07, J2 Conn_02x05_Odd_Even, J3 Conn_02x05_Odd_Even, J4 Screw_Terminal_01x02, J5 Conn_01x04_Pin, J7 Conn_01x06_Pin, J9 Jumper_Pin_ VIO_CP&3V3, P1 USB_C_Plug (Conv), P2 USB_C_Plug (Prog), SW1 SW_DIP_x02, SW2 SW_DIP_x02, SW3 SW_Push, U1 AMS1117, U2 AMS1117, U3 STM32F103CBTx, U4 CP2102N-Axx-xQFN24, Y1 8MHz

Commit message: Add files via upload
1.1.0
Parts:
- removed C20, C21, C24: 10uF, Capacitor_SMD:C_0805_2012Metric, symbol Device:C
- removed C5, C8, C9: 100nF, Capacitor_SMD:C_0805_2012Metric, symbol Device:C
- removed D10: LED_Red, LED_SMD:LED_0805_2012Metric, symbol Device:LED
- removed D16, D17: LED_Green, LED_SMD:LED_0805_2012Metric, symbol Device:LED
- removed D18: LED_Yellow, LED_SMD:LED_0805_2012Metric, symbol Device:LED
- removed D3, D4, D5, D6: PESD3V3S2UAT,215, Lt_Dev:SOT95P230X110-3N, symbol PESD3V3S2UAT_215:PESD3V3S2UAT,215
- removed J2, J3: Conn_02x05_Odd_Even, Connector_PinHeader_2.54mm:PinHeader_2x05_P2.54mm_Vertical_SMD, symbol Connector_Generic:Conn_02x05_Odd_Even
- removed J5: Conn_01x04_Pin, Connector_PinHeader_2.54mm:PinHeader_2x02_P2.54mm_Vertical_SMD, symbol Connector:Conn_01x04_Pin
- removed J7: Conn_01x06_Pin, Connector_PinHeader_2.54mm:PinHeader_2x03_P2.54mm_Vertical_SMD, symbol Connector:Conn_01x06_Pin
- removed J9: Jumper_Pin_ VIO_CP&3V3, Connector_PinHeader_2.54mm:PinHeader_1x03_P2.54mm_Vertical_SMD_Pin1Left, symbol Connector:Conn_01x03_Pin
- removed R19, R20: 100R, Resistor_SMD:R_0805_2012Metric, symbol Device:R
- removed R25: 220R, Resistor_SMD:R_0805_2012Metric, symbol Device:R
- added C32: 100nF, Capacitor_SMD:C_0805_2012Metric, symbol Device:C
- added C33: 4.7uF, Capacitor_SMD:C_0805_2012Metric, symbol Device:C
- added D11, D19, D20, D21: LED_Red, LED_SMD:LED_0805_2012Metric, symbol Device:LED
- added D22: CMS04_TE12L,Q,M_, Lt_Dev:SODFL4724X108N, symbol CMS04_TE12L_Q_M_:CMS04_TE12L,Q,M_
- added D23, D24, D25, D26, D3, D4, D5, D6: SLVU2.8-MS, Package_TO_SOT_SMD:SOT-23, symbol Diode:BAV70
- added D28, D29, D30, D31: LED_Green, LED_SMD:LED_0805_2012Metric, symbol Device:LED
- added IC5: TS3A4742DCNR, Lt_Dev:SOT65P280X145-8N, symbol TS3A4742DCNR:TS3A4742DCNR
- added IC6, IC7, IC8: TS3A4741DCNR, Lt_Dev:SOT65P280X145-8N, symbol TS3A4741DCNR:TS3A4741DCNR
- added J2, J3: Conn_JTAG_02x07, Connector_PinHeader_2.54mm:PinHeader_2x07_P2.54mm_Vertical_SMD, symbol Connector_Generic:Conn_02x07_Odd_Even
- added J5, J6, J7: Conn_02x02_Odd_Even, Connector_PinSocket_2.54mm:PinSocket_2x02_P2.54mm_Vertical_SMD, symbol Connector_Generic:Conn_02x02_Odd_Even
- added R35, R36, R37: 120R, Resistor_SMD:R_0805_2012Metric, symbol Device:R
- added R38, R40, R41, R42, R43: 100R, Resistor_SMD:R_0805_2012Metric, symbol Device:R
- C4: value 100nF -> 4.7uF
- D9: value LED_Red -> LED_Yellow
- J1: footprint Connector_PinHeader_2.54mm:PinHeader_2x07_P2.54mm_Vertical_SMD -> Connector_PinHeader_1.27mm:PinHeader_2x07_P1.27mm_Vertical_SMD
- R29: value 2k -> 1k
- renumbered D11 to D10
Connections:
- net 3V3_USB1: now also D12.2 (A), D13.2 (A), D28.2 (A), D29.2 (A), D30.2 (A), D31.2 (A), IC6.2 (VCC), IC7.2 (VCC), IC8.2 (VCC), J6.3 (Pin_3); no longer C3.1, C4.1, C7.1, IC1.16 (VDD), R2.1, R3.1, U4.6 (VDD)
- net 3V3_USB2: now also D14.2 (A), D15.2 (A), IC5.2 (VCC), J2.1 (Pin_1), J5.2 (Pin_2)
- net 5V_USB1: now also C32.2, C33.2, J6.1 (Pin_1)
- net 5V_USB2: now also J5.4 (Pin_4)
- net 5V_VTB: now also R35.2
- net B0: now also J2.5 (Pin_5)
- net CLK: now also J2.7 (Pin_7)
- net CTS: now also J3.5 (Pin_5)
- net DCD: now also J3.6 (Pin_6)
- net DIO: now also J2.9 (Pin_9)
- net DSR: now also J3.10 (Pin_10)
- net DTR: now also J3.8 (Pin_8)
- net GND: now also C3.2, C4.2, R1.1, C32.1, C33.1, D19.1 (K), D20.1 (K), D21.1 (K), D23.1 (A), D23.2 (A), D24.1 (A), D24.2 (A), D25.1 (A), D25.2 (A), D26.1 (A), D26.2 (A), D3.1 (A), D3.2 (A), D4.1 (A), D4.2 (A), D5.1 (A), D5.2 (A), D6.1 (A), D6.2 (A), IC5.4 (COM2), IC5.5 (GND), IC5.7 (COM1), IC6.4 (COM2), IC6.5 (GND), IC6.7 (COM1), IC7.4 (COM2), IC7.5 (GND), IC7.7 (COM1), IC8.4 (COM2), IC8.5 (GND), IC8.7 (COM1), J2.12 (Pin_12), J3.14 (Pin_14), J5.1 (Pin_1), J5.3 (Pin_3), J6.2 (Pin_2), J6.4 (Pin_4), J7.3 (Pin_3); no longer D12.1 (K), D13.1 (K), D14.1 (K), D15.1 (K), IC1.1 (SEL1), IC1.10 (SEL2), IC1.11 (SEL3), IC1.20 (SEL4)
- net GPIO.0: now also J3.7 (Pin_7)
- net GPIO.1: now also J3.9 (Pin_9)
- net GPIO.2: now also J3.11 (Pin_11)
- net GPIO.3: now also J3.13 (Pin_13)
- net JTAG_CLK: now also SW2.3, D6.3 (K), IC5.1 (IN1), J7.4 (Pin_4); no longer SW2.4
- net JTAG_DIO: now also SW2.4, D26.3 (K), IC5.6 (IN2), J7.2 (Pin_2); no longer SW2.3
- net LED: now also D11.2 (A)
- net RENUM: now also J2.3 (Pin_3)
- net RTS: now also J3.3 (Pin_3)
- net RXD: now also J3.1 (Pin_1)
- net RX_GPS: now also D5.3 (K), IC7.1 (IN1); no longer R16.2
- net RX_XBEE: now also D23.3 (K), IC8.1 (IN1); no longer R18.2
- net RX_uC: now also D3.3 (K), IC6.1 (IN1)
- net TXD: now also J3.12 (Pin_12)
- net TX_GPS: now also D25.3 (K), IC7.6 (IN2); no longer R15.2
- net TX_XBEE: now also D24.3 (K), IC8.6 (IN2); no longer R17.2
- net TX_uC: now also D4.3 (K), IC6.6 (IN2)
- net T_CLK: now also SW2.2, J2.8 (Pin_8); no longer SW2.1
- net T_DIO: now also SW2.1, J2.13 (Pin_13); no longer SW2.2
- net T_RST: now also J2.10 (Pin_10)
- net T_RX: now also J2.6 (Pin_6)
- net T_SWO: now also J2.11 (Pin_11)
- net T_TX: now also J2.4 (Pin_4)
- net VIO_CP: now also C3.1, C4.1, U4.6 (VDD), J3.4 (Pin_4)
- net VOUT: now also D22.2 (A), R37.2; no longer J1.3 (Pin_3)
- net VTPS: now also R36.2
- net nSUSPEND: now also R38.2
- net at R18.1: now also D15.1 (K); no longer D15.2 (A)
- net at R15.1: now also D12.1 (K); no longer D12.2 (A)
- net at R16.1: now also D13.1 (K); no longer D13.2 (A)
- net SW1_DIP2: now reaches R2.2, SW1.3
- net SW1_DIP2: now also IC1.11 (SEL3), IC1.20 (SEL4)
- net 3V3_target: now reaches J1.5 (Pin_5)
- net 3V3_target: now also C7.1, IC1.16 (VDD), R2.1, R3.1, J2.14 (Pin_14), J7.1 (Pin_1)
- net at R23.2: now also D11.1 (K)
- net at D9.2 (A): now also R38.1; no longer R1.1
- net SW1_DIP1: now reaches R3.2, SW1.4
- net SW1_DIP1: now also IC1.1 (SEL1), IC1.10 (SEL2)
- net at R17.1: now also D14.1 (K); no longer D14.2 (A)
- net NRST renamed NRST_uC
- net NRST_uC: now also J2.2 (Pin_2)
- net RI renamed RI_CLK
- net RI_CLK: now also J3.2 (Pin_2)
- new net: IC7.3 (NO2), R40.2
- new net: IC7.8 (NO1), R41.2
- new net: D29.1 (K), R41.1
- new net: D28.1 (K), R40.1
- new net: IC5.3 (NC2), R17.2
- new net: IC5.8 (NC1), R18.2
- new net: D31.1 (K), R43.1
- new net: IC8.8 (NO1), R43.2
- new net: IC6.3 (NO2), R15.2
- new net: D30.1 (K), R42.1
- new net: IC6.8 (NO1), R16.2
- new net: D20.2 (A), R36.1
- new net: D21.2 (A), R37.1
- new net: IC8.3 (NO2), R42.2
- new net: D19.2 (A), R35.1
- new net VOUT_JTAG: D22.1 (K), J1.3 (Pin_3)
Other:
- note removed: "???"
- moved on the sheet: C1, C11, C16, C17, C18, C19, C2, C22, C23, C25, C26, C27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

Commit message: Add files via upload
Parts:
- J5, J6, J7: footprint Connector_PinSocket_2.54mm:PinSocket_2x02_P2.54mm_Vertical_SMD -> Connector_PinHeader_2.54mm:PinHeader_2x02_P2.54mm_Vertical_SMD
Changed lines of the file:
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@@
       (effects (font (size 1.27 1.27)))
     )
-    (property "Footprint" "Connector_PinSocket_2.54mm:PinSocket_2x02_P2.54mm_Vertical_SMD" (at 111.76 106.045 0)
+    (property "Footprint" "Connector_PinHeader_2.54mm:PinHeader_2x02_P2.54mm_Vertical_SMD" (at 111.76 106.045 0)
       (effects (font (size 1.27 1.27)) hide)
     )
@@
       (effects (font (size 1.27 1.27)))
     )
-    (property "Footprint" "Connector_PinSocket_2.54mm:PinSocket_2x02_P2.54mm_Vertical_SMD" (at 252.73 167.64 0)
+    (property "Footprint" "Connector_PinHeader_2.54mm:PinHeader_2x02_P2.54mm_Vertical_SMD" (at 252.73 167.64 0)
       (effects (font (size 1.27 1.27)) hide)
     )
@@
       (effects (font (size 1.27 1.27)))
     )
-    (property "Footprint" "Connector_PinSocket_2.54mm:PinSocket_2x02_P2.54mm_Vertical_SMD" (at 365.125 135.255 0)
+    (property "Footprint" "Connector_PinHeader_2.54mm:PinHeader_2x02_P2.54mm_Vertical_SMD" (at 365.125 135.255 0)
       (effects (font (size 1.27 1.27)) hide)
     )

Commit message: v.1.1.2
Parts:
- removed SW1, SW2: SW_DIP_x02, Button_Switch_SMD:SW_DIP_SPSTx02_Slide_Copal_CHS-02A_W5.08mm_P1.27mm_JPin, symbol Switch:SW_DIP_x02
- added SW1, SW2: DSHP02TSGER, Lt_Dev:DSHP02TSGER, symbol DSHP02TSGER:DSHP02TSGER
Connections:
- net 3V3_USB1: now also J6.1 (Pin_1); no longer J6.3 (Pin_3)
- net 3V3_USB2: now also J5.4 (Pin_4); no longer J5.2 (Pin_2)
- net 3V3_target: now also J7.3 (Pin_3); no longer J7.1 (Pin_1)
- net 5V_USB1: now also J6.3 (Pin_3); no longer J6.1 (Pin_1)
- net 5V_USB2: now also J5.2 (Pin_2); no longer J5.4 (Pin_4)
- net GND: now also J7.1 (Pin_1), SW1.1P1, SW1.2P1; no longer J7.3 (Pin_3)
- net JTAG_CLK: now also J7.2 (Pin_2), SW2.2P2; no longer J7.4 (Pin_4)
- net JTAG_DIO: now also J7.4 (Pin_4), SW2.1P2; no longer J7.2 (Pin_2)
- net SW1_DIP1: now also SW1.1P2
- net SW1_DIP2: now also SW1.2P2
- net T_CLK: now also SW2.2P1
- net T_DIO: now also SW2.1P1
